Commit message: The force and torque was corrected to the value around the center of mass axis

File: choreonoid_ros/model/box04.urdf (robot description, URDF)
Before this commit: robot box100x100x100_1Kg, 1 links, 0 joints
Links:
- removed link BOX01KG
- added link BOX04, mass 1.0; collision box size=1.0 1.0 1.0; visual box size=1.0 1.0 1.0
